File: inprot.sch (KiCad schematic (older format))
At the start: 3 parts

Commit message: cambios varios, agregado esp-12e
Other:
- moved on the sheet: D15, R23, R24
Changed lines of the file:
@@
 $Descr A4 11693 8268
 encoding utf-8
-Sheet 13 21
-Title "Input Protection"
-Date "2021-06-10"
+Sheet 8 9
+Title "PowerMike"
+Date "2021-09-26"
 Rev "0.1"
 Comp ""
-Comment1 "https://github.com/enriquewph/esp32-ups-monitor"
+Comment1 "https://github.com/enriquewph/PowerMike"
 Comment2 ""
 Comment3 ""
@@
 L Diode:BAT54S D9
 U 1 1 60E60B36
-P 6000 3150
+P 5700 3900
 AR Path="/60E45CE9/60E60B36" Ref="D9"  Part="1"
 AR Path="/61276139/60E60B36" Ref="D14"  Part="1"
 AR Path="/612F6239/60E60B36" Ref="D15"  Part="1"
 AR Path="/6132323D/60E60B36" Ref="D16"  Part="1"
-F 0 "D16" V 6046 3238 50  0000 L CNN
-F 1 "BAT54S" V 5955 3238 50  0000 L CNN
-F 2 "Package_TO_SOT_SMD:SOT-23" H 6075 3275 50  0001 L CNN
-F 3 "https://rocelec.widen.net/view/pdf/gyex6hm7nf/PHGLS25648-1.pdf?t.download=true&u=5oefqw" H 5880 3150 50  0001 C CNN
-F 4 "BAT54S,215" H 6000 3150 50  0001 C CNN "manf#"
-	1    6000 3150
+F 0 "D15" V 5746 3988 50  0000 L CNN
+F 1 "BAT54S" V 5655 3988 50  0000 L CNN
+F 2 "Package_TO_SOT_SMD:SOT-23" H 5775 4025 50  0001 L CNN
+F 3 "https://rocelec.widen.net/view/pdf/gyex6hm7nf/PHGLS25648-1.pdf?t.download=true&u=5oefqw" H 5580 3900 50  0001 C CNN
+F 4 "BAT54S,215" H 5700 3900 50  0001 C CNN "manf#"
+	1    5700 3900
 	0    1    -1   0
 $EndComp
@@
 L Device:R R18
 U 1 1 60E62337
-P 5550 3600
+P 5250 4350
 AR Path="/60E45CE9/60E62337" Ref="R18"  Part="1"
 AR Path="/61276139/60E62337" Ref="R21"  Part="1"
 AR Path="/612F6239/60E62337" Ref="R23"  Part="1"
 AR Path="/6132323D/60E62337" Ref="R25"  Part="1"
-F 0 "R25" V 5450 3500 50  0000 C CNN
-F 1 "1k" V 5450 3650 50  0000 C CNN
-F 2 "Resistor_SMD:R_1206_3216Metric" V 5480 3600 50  0001 C CNN
-F 3 "https://www.yageo.com/upload/media/product/productsearch/datasheet/rchip/PYu-RC_Group_51_RoHS_L_11.pdf" H 5550 3600 50  0001 C CNN
-F 4 "RC1206FR-071KL" H 5550 3600 50  0001 C CNN "manf#"
-	1    5550 3600
+F 0 "R23" V 5150 4250 50  0000 C CNN
+F 1 "1k" V 5150 4400 50  0000 C CNN
+F 2 "Resistor_SMD:R_1206_3216Metric" V 5180 4350 50  0001 C CNN
+F 3 "https://www.yageo.com/upload/media/product/productsearch/datasheet/rchip/PYu-RC_Group_51_RoHS_L_11.pdf" H 5250 4350 50  0001 C CNN
+F 4 "RC1206FR-071KL" H 5250 4350 50  0001 C CNN "manf#"
+	1    5250 4350
 	0    1    1    0
 $EndComp
@@
 L Device:R R19
 U 1 1 60E62A46
-P 6400 3600
+P 6100 4350
 AR Path="/60E45CE9/60E62A46" Ref="R19"  Part="1"
 AR Path="/61276139/60E62A46" Ref="R22"  Part="1"
 AR Path="/612F6239/60E62A46" Ref="R24"  Part="1"
 AR Path="/6132323D/60E62A46" Ref="R26"  Part="1"
-F 0 "R26" V 6300 3500 50  0000 C CNN
-F 1 "1k" V 6300 3650 50  0000 C CNN
-F 2 "Resistor_SMD:R_1206_3216Metric" V 6330 3600 50  0001 C CNN
-F 3 "https://www.yageo.com/upload/media/product/productsearch/datasheet/rchip/PYu-RC_Group_51_RoHS_L_11.pdf" H 6400 3600 50  0001 C CNN
-F 4 "RC1206FR-071KL" H 6400 3600 50  0001 C CNN "manf#"
-	1    6400 3600
+F 0 "R24" V 6000 4250 50  0000 C CNN
+F 1 "1k" V 6000 4400 50  0000 C CNN
+F 2 "Resistor_SMD:R_1206_3216Metric" V 6030 4350 50  0001 C CNN
+F 3 "https://www.yageo.com/upload/media/product/productsearch/datasheet/rchip/PYu-RC_Group_51_RoHS_L_11.pdf" H 6100 4350 50  0001 C CNN
+F 4 "RC1206FR-071KL" H 6100 4350 50  0001 C CNN "manf#"
+	1    6100 4350
 	0    1    1    0
 $EndComp
@@
 L power:GND #PWR055
 U 1 1 60E632B2
-P 6000 3750
+P 5700 4500
 AR Path="/60E45CE9/60E632B2" Ref="#PWR055"  Part="1"
 AR Path="/61276139/60E632B2" Ref="#PWR0130"  Part="1"
 AR Path="/612F6239/60E632B2" Ref="#PWR0136"  Part="1"
 AR Path="/6132323D/60E632B2" Ref="#PWR0142"  Part="1"
-F 0 "#PWR0142" H 6000 3500 50  0001 C CNN
-F 1 "GND" H 6005 3577 50  0000 C CNN
-F 2 "" H 6000 3750 50  0001 C CNN
-F 3 "" H 6000 3750 50  0001 C CNN
-	1    6000 3750
+F 0 "#PWR0136" H 5700 4250 50  0001 C CNN
+F 1 "GND" H 5705 4327 50  0000 C CNN
+F 2 "" H 5700 4500 50  0001 C CNN
+F 3 "" H 5700 4500 50  0001 C CNN
+	1    5700 4500
 	1    0    0    -1
 $EndComp
 Wire Wire Line
-	6000 3450 6000 3750
+	5700 4200 5700 4500
 $Comp
 L power:+3V3 #PWR054
 U 1 1 60E63A61
-P 6000 2700
+P 5700 3450
 AR Path="/60E45CE9/60E63A61" Ref="#PWR054"  Part="1"
 AR Path="/61276139/60E63A61" Ref="#PWR0131"  Part="1"
 AR Path="/612F6239/60E63A61" Ref="#PWR0137"  Part="1"
 AR Path="/6132323D/60E63A61" Ref="#PWR0143"  Part="1"
-F 0 "#PWR0143" H 6000 2550 50  0001 C CNN
-F 1 "+3V3" H 6015 2873 50  0000 C CNN
-F 2 "" H 6000 2700 50  0001 C CNN
-F 3 "" H 6000 2700 50  0001 C CNN
-	1    6000 2700
+F 0 "#PWR0137" H 5700 3300 50  0001 C CNN
+F 1 "+3V3" H 5715 3623 50  0000 C CNN
+F 2 "" H 5700 3450 50  0001 C CNN
+F 3 "" H 5700 3450 50  0001 C CNN
+	1    5700 3450
 	1    0    0    -1
 $EndComp
 Wire Wire Line
-	6000 2700 6000 2850
-Text HLabel 5300 3600 0    39   Input ~ 0
+	5700 3450 5700 3600
+Text HLabel 5000 4350 0    39   Input ~ 0
 IN
-Text HLabel 6650 3600 2    39   Output ~ 0
+Text HLabel 6350 4350 2    39   Output ~ 0
 OUT
 Wire Wire Line
-	6650 3600 6550 3600
+	6350 4350 6250 4350
 Wire Wire Line
-	6250 3600 5750 3600
+	5950 4350 5450 4350
 Wire Wire Line
-	5400 3600 5300 3600
+	5100 4350 5000 4350
 Wire Wire Line
-	5800 3150 5750 3150
+	5500 3900 5450 3900
 Wire Wire Line
-	5750 3150 5750 3600
-Connection ~ 5750 3600
+	5450 3900 5450 4350
+Connection ~ 5450 4350
 Wire Wire Line
-	5750 3600 5700 3600
+	5450 4350 5400 4350
 $EndSCHEMATC

Commit message: demasiados cambios mi loco
Parts:
- renumbered D9 to D5, R18 to R10, R19 to R11
Changed lines of the file:
@@
 $Descr A4 11693 8268
 encoding utf-8
-Sheet 8 9
+Sheet 3 5
 Title "PowerMike"
 Date "2021-09-26"
@@
 $EndDescr
 $Comp
-L Diode:BAT54S D9
+L Diode:BAT54S D?
 U 1 1 60E60B36
 P 5700 3900
-AR Path="/60E45CE9/60E60B36" Ref="D9"  Part="1"
-AR Path="/61276139/60E60B36" Ref="D14"  Part="1"
-AR Path="/612F6239/60E60B36" Ref="D15"  Part="1"
-AR Path="/6132323D/60E60B36" Ref="D16"  Part="1"
-F 0 "D15" V 5746 3988 50  0000 L CNN
+AR Path="/60E45CE9/60E60B36" Ref="D?"  Part="1"
+AR Path="/61276139/60E60B36" Ref="D?"  Part="1"
+AR Path="/612F6239/60E60B36" Ref="D5"  Part="1"
+AR Path="/6132323D/60E60B36" Ref="D?"  Part="1"
+F 0 "D5" V 5746 3988 50  0000 L CNN
 F 1 "BAT54S" V 5655 3988 50  0000 L CNN
 F 2 "Package_TO_SOT_SMD:SOT-23" H 5775 4025 50  0001 L CNN
@@
 $EndComp
 $Comp
-L Device:R R18
+L Device:R R?
 U 1 1 60E62337
 P 5250 4350
-AR Path="/60E45CE9/60E62337" Ref="R18"  Part="1"
-AR Path="/61276139/60E62337" Ref="R21"  Part="1"
-AR Path="/612F6239/60E62337" Ref="R23"  Part="1"
-AR Path="/6132323D/60E62337" Ref="R25"  Part="1"
-F 0 "R23" V 5150 4250 50  0000 C CNN
+AR Path="/60E45CE9/60E62337" Ref="R?"  Part="1"
+AR Path="/61276139/60E62337" Ref="R?"  Part="1"
+AR Path="/612F6239/60E62337" Ref="R10"  Part="1"
+AR Path="/6132323D/60E62337" Ref="R?"  Part="1"
+F 0 "R10" V 5150 4250 50  0000 C CNN
 F 1 "1k" V 5150 4400 50  0000 C CNN
 F 2 "Resistor_SMD:R_1206_3216Metric" V 5180 4350 50  0001 C CNN
@@
 $EndComp
 $Comp
-L Device:R R19
+L Device:R R?
 U 1 1 60E62A46
 P 6100 4350
-AR Path="/60E45CE9/60E62A46" Ref="R19"  Part="1"
-AR Path="/61276139/60E62A46" Ref="R22"  Part="1"
-AR Path="/612F6239/60E62A46" Ref="R24"  Part="1"
-AR Path="/6132323D/60E62A46" Ref="R26"  Part="1"
-F 0 "R24" V 6000 4250 50  0000 C CNN
+AR Path="/60E45CE9/60E62A46" Ref="R?"  Part="1"
+AR Path="/61276139/60E62A46" Ref="R?"  Part="1"
+AR Path="/612F6239/60E62A46" Ref="R11"  Part="1"
+AR Path="/6132323D/60E62A46" Ref="R?"  Part="1"
+F 0 "R11" V 6000 4250 50  0000 C CNN
 F 1 "1k" V 6000 4400 50  0000 C CNN
 F 2 "Resistor_SMD:R_1206_3216Metric" V 6030 4350 50  0001 C CNN
@@
 $EndComp
 $Comp
-L power:GND #PWR055
+L power:GND #PWR?
 U 1 1 60E632B2
 P 5700 4500
-AR Path="/60E45CE9/60E632B2" Ref="#PWR055"  Part="1"
-AR Path="/61276139/60E632B2" Ref="#PWR0130"  Part="1"
-AR Path="/612F6239/60E632B2" Ref="#PWR0136"  Part="1"
-AR Path="/6132323D/60E632B2" Ref="#PWR0142"  Part="1"
-F 0 "#PWR0136" H 5700 4250 50  0001 C CNN
+AR Path="/60E45CE9/60E632B2" Ref="#PWR?"  Part="1"
+AR Path="/61276139/60E632B2" Ref="#PWR?"  Part="1"
+AR Path="/612F6239/60E632B2" Ref="#PWR046"  Part="1"
+AR Path="/6132323D/60E632B2" Ref="#PWR?"  Part="1"
+F 0 "#PWR046" H 5700 4250 50  0001 C CNN
 F 1 "GND" H 5705 4327 50  0000 C CNN
 F 2 "" H 5700 4500 50  0001 C CNN
@@
 	5700 4200 5700 4500
 $Comp
-L power:+3V3 #PWR054
+L power:+3V3 #PWR?
 U 1 1 60E63A61
 P 5700 3450
-AR Path="/60E45CE9/60E63A61" Ref="#PWR054"  Part="1"
-AR Path="/61276139/60E63A61" Ref="#PWR0131"  Part="1"
-AR Path="/612F6239/60E63A61" Ref="#PWR0137"  Part="1"
-AR Path="/6132323D/60E63A61" Ref="#PWR0143"  Part="1"
-F 0 "#PWR0137" H 5700 3300 50  0001 C CNN
+AR Path="/60E45CE9/60E63A61" Ref="#PWR?"  Part="1"
+AR Path="/61276139/60E63A61" Ref="#PWR?"  Part="1"
+AR Path="/612F6239/60E63A61" Ref="#PWR045"  Part="1"
+AR Path="/6132323D/60E63A61" Ref="#PWR?"  Part="1"
+F 0 "#PWR045" H 5700 3300 50  0001 C CNN
 F 1 "+3V3" H 5715 3623 50  0000 C CNN
 F 2 "" H 5700 3450 50  0001 C CNN
