File: lm35.sch (KiCad schematic (older format))
At the start: 3 parts, among them J7 Conn_01x03

Commit message: cambios varios, agregado esp-12e
Changed lines of the file:
@@
 $Descr A4 11693 8268
 encoding utf-8
-Sheet 10 21
-Title "Temperature Sensor Input"
-Date "2021-06-10"
+Sheet 7 9
+Title "PowerMike"
+Date "2021-09-26"
 Rev "0.1"
 Comp ""
-Comment1 "https://github.com/enriquewph/esp32-ups-monitor"
+Comment1 "https://github.com/enriquewph/PowerMike"
 Comment2 ""
 Comment3 ""
@@
 AR Path="/612F4D6E/61313C16" Ref="J7"  Part="1"
 AR Path="/61323238/61313C16" Ref="J8"  Part="1"
-F 0 "J8" H 4800 3200 50  0000 L CNN
+F 0 "J7" H 4800 3200 50  0000 L CNN
 F 1 "Conn_01x03" H 4930 2901 50  0001 L CNN
 F 2 "Connector_Molex:Molex_KK-254_AE-6410-03A_1x03_P2.54mm_Vertical" H 4850 2950 50  0001 C CNN
@@
 AR Path="/612F4D6E/61313C25" Ref="#PWR0132"  Part="1"
 AR Path="/61323238/61313C25" Ref="#PWR0138"  Part="1"
-F 0 "#PWR0138" H 5850 2600 50  0001 C CNN
+F 0 "#PWR0132" H 5850 2600 50  0001 C CNN
 F 1 "+3V3" H 5865 2923 50  0000 C CNN
 F 2 "" H 5850 2750 50  0001 C CNN
@@
 AR Path="/612F4D6E/61313C2B" Ref="#PWR0133"  Part="1"
 AR Path="/61323238/61313C2B" Ref="#PWR0139"  Part="1"
-F 0 "#PWR0139" H 5350 3200 50  0001 C CNN
+F 0 "#PWR0133" H 5350 3200 50  0001 C CNN
 F 1 "GND" H 5355 3277 50  0000 C CNN
 F 2 "" H 5350 3450 50  0001 C CNN
@@
 AR Path="/612F4D6E/61313C31" Ref="#PWR0134"  Part="1"
 AR Path="/61323238/61313C31" Ref="#PWR0140"  Part="1"
-F 0 "#PWR0140" H 5150 3200 50  0001 C CNN
+F 0 "#PWR0134" H 5150 3200 50  0001 C CNN
 F 1 "GND" H 5155 3277 50  0000 C CNN
 F 2 "" H 5150 3450 50  0001 C CNN
@@
 AR Path="/612F4D6E/61316DCA" Ref="C18"  Part="1"
 AR Path="/61323238/61316DCA" Ref="C20"  Part="1"
-F 0 "C20" H 5465 3246 50  0000 L CNN
+F 0 "C18" H 5465 3246 50  0000 L CNN
 F 1 "100nF" H 5465 3155 50  0000 L CNN
 F 2 "Capacitor_SMD:C_1206_3216Metric_Pad1.33x1.80mm_HandSolder" H 5388 3050 50  0001 C CNN
@@
 AR Path="/612F4D6E/613172F1" Ref="#PWR0135"  Part="1"
 AR Path="/61323238/613172F1" Ref="#PWR0141"  Part="1"
-F 0 "#PWR0141" H 5850 3200 50  0001 C CNN
+F 0 "#PWR0135" H 5850 3200 50  0001 C CNN
 F 1 "GND" H 5855 3277 50  0000 C CNN
 F 2 "" H 5850 3450 50  0001 C CNN
@@
 AR Path="/612F4D6E/613172FB" Ref="C19"  Part="1"
 AR Path="/61323238/613172FB" Ref="C21"  Part="1"
-F 0 "C21" H 5965 3246 50  0000 L CNN
+F 0 "C19" H 5965 3246 50  0000 L CNN
 F 1 "100nF" H 5965 3155 50  0000 L CNN
 F 2 "Capacitor_SMD:C_1206_3216Metric_Pad1.33x1.80mm_HandSolder" H 5888 3050 50  0001 C CNN

Commit message: demasiados cambios mi loco
Parts:
- renumbered C18 to C11, C19 to C12, J7 to J5
Changed lines of the file:
@@
 $Descr A4 11693 8268
 encoding utf-8
-Sheet 7 9
+Sheet 7 5
 Title "PowerMike"
 Date "2021-09-26"
@@
 P 4850 2950
 AR Path="/61313C16" Ref="J?"  Part="1"
-AR Path="/612F4D6E/61313C16" Ref="J7"  Part="1"
-AR Path="/61323238/61313C16" Ref="J8"  Part="1"
-F 0 "J7" H 4800 3200 50  0000 L CNN
+AR Path="/612F4D6E/61313C16" Ref="J5"  Part="1"
+AR Path="/61323238/61313C16" Ref="J?"  Part="1"
+F 0 "J5" H 4800 3200 50  0000 L CNN
 F 1 "Conn_01x03" H 4930 2901 50  0001 L CNN
 F 2 "Connector_Molex:Molex_KK-254_AE-6410-03A_1x03_P2.54mm_Vertical" H 4850 2950 50  0001 C CNN
@@
 P 5850 2750
 AR Path="/61313C25" Ref="#PWR?"  Part="1"
-AR Path="/612F4D6E/61313C25" Ref="#PWR0132"  Part="1"
-AR Path="/61323238/61313C25" Ref="#PWR0138"  Part="1"
-F 0 "#PWR0132" H 5850 2600 50  0001 C CNN
+AR Path="/612F4D6E/61313C25" Ref="#PWR043"  Part="1"
+AR Path="/61323238/61313C25" Ref="#PWR?"  Part="1"
+F 0 "#PWR043" H 5850 2600 50  0001 C CNN
 F 1 "+3V3" H 5865 2923 50  0000 C CNN
 F 2 "" H 5850 2750 50  0001 C CNN
@@
 P 5350 3450
 AR Path="/61313C2B" Ref="#PWR?"  Part="1"
-AR Path="/612F4D6E/61313C2B" Ref="#PWR0133"  Part="1"
-AR Path="/61323238/61313C2B" Ref="#PWR0139"  Part="1"
-F 0 "#PWR0133" H 5350 3200 50  0001 C CNN
+AR Path="/612F4D6E/61313C2B" Ref="#PWR042"  Part="1"
+AR Path="/61323238/61313C2B" Ref="#PWR?"  Part="1"
+F 0 "#PWR042" H 5350 3200 50  0001 C CNN
 F 1 "GND" H 5355 3277 50  0000 C CNN
 F 2 "" H 5350 3450 50  0001 C CNN
@@
 P 5150 3450
 AR Path="/61313C31" Ref="#PWR?"  Part="1"
-AR Path="/612F4D6E/61313C31" Ref="#PWR0134"  Part="1"
-AR Path="/61323238/61313C31" Ref="#PWR0140"  Part="1"
-F 0 "#PWR0134" H 5150 3200 50  0001 C CNN
+AR Path="/612F4D6E/61313C31" Ref="#PWR041"  Part="1"
+AR Path="/61323238/61313C31" Ref="#PWR?"  Part="1"
+F 0 "#PWR041" H 5150 3200 50  0001 C CNN
 F 1 "GND" H 5155 3277 50  0000 C CNN
 F 2 "" H 5150 3450 50  0001 C CNN
@@
 $EndComp
 $Comp
-L Device:C C18
+L Device:C C11
 U 1 1 61316DCA
 P 5350 3200
-AR Path="/612F4D6E/61316DCA" Ref="C18"  Part="1"
-AR Path="/61323238/61316DCA" Ref="C20"  Part="1"
-F 0 "C18" H 5465 3246 50  0000 L CNN
+AR Path="/612F4D6E/61316DCA" Ref="C11"  Part="1"
+AR Path="/61323238/61316DCA" Ref="C?"  Part="1"
+F 0 "C11" H 5465 3246 50  0000 L CNN
 F 1 "100nF" H 5465 3155 50  0000 L CNN
 F 2 "Capacitor_SMD:C_1206_3216Metric_Pad1.33x1.80mm_HandSolder" H 5388 3050 50  0001 C CNN
@@
 P 5850 3450
 AR Path="/613172F1" Ref="#PWR?"  Part="1"
-AR Path="/612F4D6E/613172F1" Ref="#PWR0135"  Part="1"
-AR Path="/61323238/613172F1" Ref="#PWR0141"  Part="1"
-F 0 "#PWR0135" H 5850 3200 50  0001 C CNN
+AR Path="/612F4D6E/613172F1" Ref="#PWR044"  Part="1"
+AR Path="/61323238/613172F1" Ref="#PWR?"  Part="1"
+F 0 "#PWR044" H 5850 3200 50  0001 C CNN
 F 1 "GND" H 5855 3277 50  0000 C CNN
 F 2 "" H 5850 3450 50  0001 C CNN
@@
 $EndComp
 $Comp
-L Device:C C19
+L Device:C C12
 U 1 1 613172FB
 P 5850 3200
-AR Path="/612F4D6E/613172FB" Ref="C19"  Part="1"
-AR Path="/61323238/613172FB" Ref="C21"  Part="1"
-F 0 "C19" H 5965 3246 50  0000 L CNN
+AR Path="/612F4D6E/613172FB" Ref="C12"  Part="1"
+AR Path="/61323238/613172FB" Ref="C?"  Part="1"
+F 0 "C12" H 5965 3246 50  0000 L CNN
 F 1 "100nF" H 5965 3155 50  0000 L CNN
 F 2 "Capacitor_SMD:C_1206_3216Metric_Pad1.33x1.80mm_HandSolder" H 5888 3050 50  0001 C CNN
