File: psu.sch (KiCad schematic (older format))
At the start: 17 parts, among them U7 LM2596S-3.3, U9 AMS1117-5.0

Commit message: demasiados cambios mi loco
Parts:
- removed C11, C12, C8, C9: 470uF, libs:CAP_10x10_SMD_THT, symbol Device:CP
- removed D7: SS14, Diode_SMD:D_SMA_Handsoldering, symbol Diode:1N5822
- removed JP1: SolderJumper_2_Open, Jumper:SolderJumper-2_P1.3mm_Open_RoundedPad1.0x1.5mm, symbol Jumper:SolderJumper_2_Open
- removed L1: 68uH, libs:L_12x12mm_H8mm, symbol Device:L
- removed R17: 330, Resistor_SMD:R_1206_3216Metric, symbol Device:R
- removed RV1: 10k, Potentiometer_THT:Potentiometer_Bourns_3296W_Vertical, symbol Device:R_POT
- removed U7: LM2596S-3.3, libs:TO-263-5_TabPin3, symbol Regulator_Switching:LM2596S-3.3
- removed U9: AMS1117-5.0, Package_TO_SOT_SMD:SOT-223-3_TabPin2, symbol Regulator_Linear:AMS1117-5.0
- added C10: 470uF, libs:CAP_10x10_SMD_THT, symbol Device:CP
- added C8: 100nF, Capacitor_SMD:C_1206_3216Metric_Pad1.33x1.80mm_HandSolder, symbol Device:C
- added D1: MB6S, Package_TO_SOT_SMD:TO-269AA, symbol Diode_Bridge:MB6S
- added J4: Screw_Terminal_01x02, libs:TerminalBlock_bornier-2_P5.08mm, symbol Connector:Screw_Terminal_01x02
- added U4: KF33BD-TR, Package_SO:SO-8_3.9x4.9mm_P1.27mm, symbol kf33:KF33BD-TR
- added U5: KF50BD-TR, Package_SO:SO-8_3.9x4.9mm_P1.27mm, symbol kf33:KF33BD-TR
- C5: Fitted No -> (none)
- renumbered C10 to C9, D6 to D2, R16 to R7
Connections:
- net GND: now also C10.2, C8.2, D1.4 (-), U4.2 (GND), U4.3 (GND), U4.5 (INH), U4.6 (GND), U4.7 (GND), U5.2 (GND), U5.3 (GND), U5.5 (INH), U5.6 (GND), U5.7 (GND)
- net VOUT: now also U4.1 (VOUT)
- net VOUT_5V: now also C10.1, U5.1 (VOUT)
- net VIN: no longer names the net of C5.1, C6.1, C7.1, D2.2 (A)
- net VIN: now also C8.1, D1.3 (+), U4.8 (VIN), U5.8 (VIN)
- new net: D1.2 (~~), J4.1 (Pin_1)
- new net: D1.1 (~~), J4.2 (Pin_2)
Other:
- note removed: "*Extra power rail for some sensors. Not needed."
- note removed: "*Recommended. Not needed."
- note removed: "*Recommended. \nNot needed."
- note removed: "Compatible with LM2575\nLM2576, LM2596S, Select \ninductor accordingly."
- note removed: "For 3.3V Version:\n- Solder JP1"
- note removed: "For 5.0V/12V\n- Solder RV1\n- Adjust until 3.3v\n- Solder remaining components."
- note removed: "For ADJ Version:\n- Solder R17\n- Solder RV1\n- Adjust until 3.3v\n- Solder remaining components."
- moved on the sheet: C6, C7, C9, D2, R7
