File: relay.sch (KiCad schematic (older format))
At the start: 6 parts, among them K1 RELAY, Q1 BC817

Commit message: demasiados cambios mi loco
Parts:
- K1: value RELAY -> RELAY 0510; manf# G5LE-1-VDDC12 -> RAS0510
- R8: renamed from R3; value 1k -> 220; manf# RC1206FR-071KL -> RC1206FR-07220RL
- renumbered D5 to D3, D8 to D4, R4 to R9
Connections:
- net +12V renamed +5V
Changed lines of the file:
@@
 $Descr A4 11693 8268
 encoding utf-8
-Sheet 6 9
+Sheet 3 5
 Title "PowerMike"
 Date "2021-09-26"
@@
 AR Path="/61070A3B" Ref="Q?"  Part="1"
 AR Path="/6102C68D/61070A3B" Ref="Q1"  Part="1"
-AR Path="/610A0B30/61070A3B" Ref="Q2"  Part="1"
-AR Path="/610C441E/61070A3B" Ref="Q3"  Part="1"
-F 0 "Q3" H 5641 4646 50  0000 L CNN
+AR Path="/610A0B30/61070A3B" Ref="Q?"  Part="1"
+AR Path="/610C441E/61070A3B" Ref="Q?"  Part="1"
+F 0 "Q1" H 5641 4646 50  0000 L CNN
 F 1 "BC817" H 5641 4555 50  0000 L CNN
 F 2 "Package_TO_SOT_SMD:SOT-23" H 5650 4525 50  0001 L CIN
@@
 P 5050 4600
 AR Path="/61070A47" Ref="R?"  Part="1"
-AR Path="/6102C68D/61070A47" Ref="R4"  Part="1"
-AR Path="/610A0B30/61070A47" Ref="R8"  Part="1"
-AR Path="/610C441E/61070A47" Ref="R10"  Part="1"
-F 0 "R10" V 4950 4500 50  0000 C CNN
+AR Path="/6102C68D/61070A47" Ref="R9"  Part="1"
+AR Path="/610A0B30/61070A47" Ref="R?"  Part="1"
+AR Path="/610C441E/61070A47" Ref="R?"  Part="1"
+F 0 "R9" V 4950 4500 50  0000 C CNN
 F 1 "1k" V 4950 4700 50  0000 C CNN
 F 2 "Resistor_SMD:R_1206_3216Metric" V 4980 4600 50  0001 C CNN
@@
 P 5550 3950
 AR Path="/61070A4D" Ref="D?"  Part="1"
-AR Path="/6102C68D/61070A4D" Ref="D8"  Part="1"
-AR Path="/610A0B30/61070A4D" Ref="D11"  Part="1"
-AR Path="/610C441E/61070A4D" Ref="D13"  Part="1"
-F 0 "D13" V 5500 3750 50  0000 L CNN
+AR Path="/6102C68D/61070A4D" Ref="D4"  Part="1"
+AR Path="/610A0B30/61070A4D" Ref="D?"  Part="1"
+AR Path="/610C441E/61070A4D" Ref="D?"  Part="1"
+F 0 "D4" V 5500 3750 50  0000 L CNN
 F 1 "M7" V 5600 3750 50  0000 L CNN
 F 2 "Diode_SMD:D_SMA_Handsoldering" H 5550 3775 50  0001 C CNN
@@
 P 5550 4850
 AR Path="/61070A53" Ref="#PWR?"  Part="1"
-AR Path="/6102C68D/61070A53" Ref="#PWR0108"  Part="1"
-AR Path="/610A0B30/61070A53" Ref="#PWR0110"  Part="1"
-AR Path="/610C441E/61070A53" Ref="#PWR0112"  Part="1"
-F 0 "#PWR0112" H 5550 4600 50  0001 C CNN
+AR Path="/6102C68D/61070A53" Ref="#PWR040"  Part="1"
+AR Path="/610A0B30/61070A53" Ref="#PWR?"  Part="1"
+AR Path="/610C441E/61070A53" Ref="#PWR?"  Part="1"
+F 0 "#PWR040" H 5550 4600 50  0001 C CNN
 F 1 "GND" H 5555 4677 50  0000 C CNN
 F 2 "" H 5550 4850 50  0001 C CNN
 F 3 "" H 5550 4850 50  0001 C CNN
 	1    5550 4850
-	1    0    0    -1
-$EndComp
-$Comp
-L power:+12V #PWR?
-U 1 1 61070A59
-P 5550 3500
-AR Path="/61070A59" Ref="#PWR?"  Part="1"
-AR Path="/6102C68D/61070A59" Ref="#PWR0109"  Part="1"
-AR Path="/610A0B30/61070A59" Ref="#PWR0111"  Part="1"
-AR Path="/610C441E/61070A59" Ref="#PWR0113"  Part="1"
-F 0 "#PWR0113" H 5550 3350 50  0001 C CNN
-F 1 "+12V" H 5565 3673 50  0000 C CNN
-F 2 "" H 5550 3500 50  0001 C CNN
-F 3 "" H 5550 3500 50  0001 C CNN
-	1    5550 3500
 	1    0    0    -1
 $EndComp
@@
 AR Path="/61070A63" Ref="K?"  Part="1"
 AR Path="/6102C68D/61070A63" Ref="K1"  Part="1"
-AR Path="/610A0B30/61070A63" Ref="K2"  Part="1"
-AR Path="/610C441E/61070A63" Ref="K3"  Part="1"
-F 0 "K3" H 6000 4200 50  0000 L CNN
-F 1 "RELAY" H 6830 3905 50  0001 L CNN
+AR Path="/610A0B30/61070A63" Ref="K?"  Part="1"
+AR Path="/610C441E/61070A63" Ref="K?"  Part="1"
+F 0 "K1" H 6000 4200 50  0000 L CNN
+F 1 "RELAY 0510" H 6830 3905 50  0001 L CNN
 F 2 "Relay_THT:Relay_SPDT_SANYOU_SRD_Series_Form_C" H 6850 3900 50  0001 L CNN
-F 3 "https://omronfs.omron.com/en_US/ecb/products/pdf/en-g5le.pdf" H 6400 3950 50  0001 C CNN
-F 4 "G5LE-1-VDDC12" H 6400 3950 50  0001 C CNN "manf#"
+F 3 "https://pdf1.alldatasheet.es/datasheet-pdf/view/1131916/SUNHOLD/RAS-0510ML1.html" H 6400 3950 50  0001 C CNN
+F 4 "RAS0510" H 6400 3950 50  0001 C CNN "manf#"
 	1    6400 3950
 	1    0    0    -1
@@
 AR Path="/6107B2AB" Ref="D?"  Part="1"
 AR Path="/60CF66AD/6107B2AB" Ref="D?"  Part="1"
-AR Path="/6102C68D/6107B2AB" Ref="D5"  Part="1"
-AR Path="/610A0B30/6107B2AB" Ref="D10"  Part="1"
-AR Path="/610C441E/6107B2AB" Ref="D12"  Part="1"
-F 0 "D12" V 4889 3632 50  0000 R CNN
+AR Path="/6102C68D/6107B2AB" Ref="D3"  Part="1"
+AR Path="/610A0B30/6107B2AB" Ref="D?"  Part="1"
+AR Path="/610C441E/6107B2AB" Ref="D?"  Part="1"
+F 0 "D3" V 4889 3632 50  0000 R CNN
 F 1 "LED" V 4798 3632 50  0000 R CNN
 F 2 "LED_SMD:LED_1206_3216Metric" H 4850 3750 50  0001 C CNN
@@
 AR Path="/6107B2B1" Ref="R?"  Part="1"
 AR Path="/60CF66AD/6107B2B1" Ref="R?"  Part="1"
-AR Path="/6102C68D/6107B2B1" Ref="R3"  Part="1"
-AR Path="/610A0B30/6107B2B1" Ref="R7"  Part="1"
-AR Path="/610C441E/6107B2B1" Ref="R9"  Part="1"
-F 0 "R9" H 4920 4196 50  0000 L CNN
-F 1 "1k" H 4920 4105 50  0000 L CNN
+AR Path="/6102C68D/6107B2B1" Ref="R8"  Part="1"
+AR Path="/610A0B30/6107B2B1" Ref="R?"  Part="1"
+AR Path="/610C441E/6107B2B1" Ref="R?"  Part="1"
+F 0 "R8" H 4920 4196 50  0000 L CNN
+F 1 "220" H 4920 4105 50  0000 L CNN
 F 2 "Resistor_SMD:R_1206_3216Metric" V 4780 4150 50  0001 C CNN
 F 3 "https://www.yageo.com/upload/media/product/productsearch/datasheet/rchip/PYu-RC_Group_51_RoHS_L_11.pdf" H 4850 4150 50  0001 C CNN
-F 4 "RC1206FR-071KL" H 4850 4150 50  0001 C CNN "manf#"
+F 4 "RC1206FR-07220RL" H 4850 4150 50  0001 C CNN "manf#"
 	1    4850 4150
 	1    0    0    -1
@@
 Wire Wire Line
 	4650 4600 4900 4600
+$Comp
+L power:+5V #PWR?
+U 1 1 617430C8
+P 5550 3500
+AR Path="/617430C8" Ref="#PWR?"  Part="1"
+AR Path="/6102C68D/617430C8" Ref="#PWR039"  Part="1"
+F 0 "#PWR039" H 5550 3350 50  0001 C CNN
+F 1 "+5V" H 5565 3673 50  0000 C CNN
+F 2 "" H 5550 3500 50  0001 C CNN
+F 3 "" H 5550 3500 50  0001 C CNN
+	1    5550 3500
+	1    0    0    -1
+$EndComp
 $EndSCHEMATC
